File: schematic/2xl.kicad_sch (KiCad schematic)
At the start: 92 parts, among them J1 eye-, J10 head+, J11 B-, J12 B+, J13 B-, J14 mouth+, J16 SP+, J17 SP-, J18 SP+, J19 SP-, J20 eye, J3 B-, J4 M-, J5 M+, J6 B+, J7 mouth-, J8 Barrel_Jack_Switch, J9 head-, Q1 9014C, Q10 9014C, Q11 S8550C, Q2 9014C, Q3 9014C, Q4 9014C, Q5 S8050D, Q6 9014C, Q7 MPSA13, Q8 9014C, Q9 9014C, SW1 Play, U1 LM386, U2 BA6220

Commit message: diodes markings
Parts:
- added J21: mouth-, symbol Connector:Conn_01x01_Pin
- added J22: mouth+, symbol Connector:Conn_01x01_Pin
- added J23, J25: eye+, symbol Connector:Conn_01x01_Pin
- added J24, J26: eye-, symbol Connector:Conn_01x01_Pin
- added LA1, LA2, LA3: Lamp, symbol Device:Lamp
- D1, D2: value D -> 1N4148
- J20: value eye -> eye+
- RV1: value R_Potentiometer -> 2K
- RV2: value R_Potentiometer -> 10K
Connections:
- new net: J26.1 (Pin_1), LA3.1 (-)
- new net: J21.1 (Pin_1), LA1.1 (-)
- new net: J22.1 (Pin_1), LA1.2 (+)
- new net: J25.1 (Pin_1), LA3.2 (+)
- new net: J24.1 (Pin_1), LA2.1 (-)
- new net: J23.1 (Pin_1), LA2.2 (+)
Other:
- moved on the sheet: BT1, C17, C18, C19, C21, C23, D3, J11, J12, J13, J14, J4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
